Commit message: Add pubs to curb detector, begin URDF adjust

File: data/voltron.urdf (robot description, URDF)
Before this commit: robot voltron, 6 links, 5 joints
Links:
- added link zed2_left_camera_optical_frame
Joints:
- added joint zed2_left_camera_optical_frame_joint: type fixed, parent base_link, child zed2_left_camera_optical_frame, origin xyz=3.4 0.0 1.0 rpy=0.0 0.0 0.0

Commit message: Recalibrate Lidar tfs (pitch and roll)

File: data/voltron.urdf (robot description, URDF)
Before this commit: robot voltron, 7 links, 6 joints
Joints:
- joint lidar_front_joint: origin xyz=3.4 -0.902 0.7876 rpy=0 0 -1.45 -> xyz=3.4 -0.902 0.7876 rpy=-0.015 -0.03 -1.45
- joint lidar_rear_joint: origin xyz=-0.1 0.9 1.0 rpy=0 -0.0672 2.65 -> xyz=-0.1 0.9 1.1 rpy=+0.03 -0.0472 2.65

Commit message: Update model in URDF

File: data/voltron.urdf (robot description, URDF)
Before this commit: robot voltron, 7 links, 6 joints
Links:
- link base_link: geometry collision box size=4.37 2.0 1.85; visual mesh filename=file:///home/main/navigator/data/hailbopp.obj scale=1.0 1.0 1.0
Joints:
- joint gnss_joint: origin xyz=0 0 0 rpy=0 0 0 -> xyz=3.4 -0.5 0.5 rpy=0 0 0

Commit message: Add IMU to state estimate

File: data/voltron.urdf (robot description, URDF)
Before this commit: robot voltron, 7 links, 6 joints
Joints:
- joint imu_joint: origin xyz=0 0 0 rpy=0 0 0 -> xyz=3.4 0.0 1.0 rpy=0 0 0

Commit message: Eh

File: data/voltron.urdf (robot description, URDF)
Before this commit: robot voltron, 7 links, 6 joints
Links:
- link base_link: geometry collision box size=4.37 2.0 1.85; visual mesh filename=file:///home/main/navigator/data/hailbopp.obj scale=1.3 1.0 1.0

Commit message: Fix road bound bl transform

File: data/voltron.urdf (robot description, URDF)
Before this commit: robot voltron, 7 links, 6 joints
Links:
- removed link nav_base
Joints:
- removed joint nav_base_joint
- joint gnss_joint: origin xyz=3.4 -0.5 0.5 rpy=0 0 0 -> xyz=0.0 -0.5 0.5 rpy=0 0 0
- joint imu_joint: origin xyz=3.4 0.0 1.0 rpy=0 0 0 -> xyz=0.0 0.0 1.0 rpy=0 0 0
- joint lidar_front_joint: origin xyz=3.4 -0.902 0.7876 rpy=-0.015 -0.03 -1.45 -> xyz=0.0 -0.902 0.7876 rpy=-0.015 -0.03 -1.45
- joint lidar_rear_joint: origin xyz=-0.1 0.9 1.1 rpy=+0.03 -0.0472 2.65 -> xyz=-3.5 0.9 1.1 rpy=+0.03 -0.0472 2.65
- joint zed2_left_camera_optical_frame_joint: origin xyz=3.4 0.0 1.0 rpy=0.0 0.0 0.0 -> xyz=0.0 0.0 1.0 rpy=0.0 0.0 0.0
