Commit message: Add "carla_lite.launch.py"

File: data/allstar.urdf (robot description, URDF)
Before this commit: robot allstar, 1 links, 1 joints
Joints:
- joint hero_to_base_link: child base_Link -> base_link

Commit message: Add GNSS-> odom conversion

File: data/allstar.urdf (robot description, URDF)
Before this commit: robot allstar, 1 links, 1 joints
Links:
- added link hero
