Commit message: Fix URDF mesh, ports, and lidar - URDF mesh now points to /home/share on Quad. 3D model works in Rviz2 - Port for CARLA now points to 2000+domain id - Domain ID of 14 => -world-port=2014 - Domain ID now passed to Docker from host on boot - Fixed error with lidar processing node - Removed one last reference to AllStar - Deleted stale 3D models from /data

File: data/carla.urdf (robot description, URDF)
Before this commit: robot carla-bopp, 2 links, 1 joints
Links:
- added link model_link; visual mesh filename=file:///home/share/hailbopp.stl scale=1.0 1.0 1.0
- link base_link: geometry collision box size=4.37 2.0 1.85
Joints:
- added joint model_joint: type fixed, parent base_link, child model_link, origin xyz=-1.7 -2.3 -0.7 rpy=0 0 -1.570796
