Commit message: Add ZED stuff

File: data/hail_bopp.urdf (robot description, URDF)
Before this commit: robot voltron, 7 links, 6 joints
Links:
- added link zed2_camera_center
Joints:
- added joint zed2_center_joint: type fixed, parent base_link, child zed2_camera_center, origin xyz=0.0 0.0 1.78 rpy=0.0 0.0 0.0

Commit message: Update URDF, add messages

File: data/hail_bopp.urdf (robot description, URDF)
Before this commit: robot voltron, 8 links, 7 joints
Links:
- removed link nav_base
Joints:
- removed joint nav_base_joint
- joint gnss_joint: origin xyz=3.4 -0.5 0.5 rpy=0 0 0 -> xyz=0.0 -0.5 0.5 rpy=0 0 0
- joint imu_joint: origin xyz=3.4 0.0 1.0 rpy=0 0 0 -> xyz=0.0 0.0 1.0 rpy=0 0 0
- joint lidar_front_joint: origin xyz=3.4 -0.902 0.7876 rpy=-0.015 -0.03 -1.45 -> xyz=0.0 -0.902 0.7876 rpy=-0.015 -0.03 -1.45
- joint lidar_rear_joint: origin xyz=-0.1 0.9 1.1 rpy=+0.03 -0.0472 2.65 -> xyz=-3.5 0.9 1.1 rpy=+0.03 -0.0472 2.65

Commit message: Fix launch transforms

File: data/hail_bopp.urdf (robot description, URDF)
Before this commit: robot voltron, 8 links, 7 joints
Links:
- removed link odom
Joints:
- removed joint temp_join

Commit message: Add IMU parsing from serial

File: data/hail_bopp.urdf (robot description, URDF)
Before this commit: robot voltron, 7 links, 6 joints
Links:
- added link arduino_imu
Joints:
- joint imu_joint: child imu -> arduino_imu; origin xyz=0.0 0.0 1.0 rpy=0 0 0 -> xyz=0.3 0.0 0.0 rpy=0 0 0

Commit message: Campus testing

File: data/hail_bopp.urdf (robot description, URDF)
Before this commit: robot voltron, 8 links, 6 joints
Joints:
- added joint arduino_imu_joint: type fixed, parent base_link, child arduino_imu, origin xyz=0.3 0.0 0.0 rpy=0 0 0
- joint imu_joint: child arduino_imu -> imu; origin xyz=0.3 0.0 0.0 rpy=0 0 0 -> xyz=0.0 0.0 1.0 rpy=0 0 0

Commit message: Remove FastGICP

File: data/hail_bopp.urdf (robot description, URDF)
Before this commit: robot voltron, 8 links, 7 joints
Links:
- link base_link: geometry collision box size=4.37 2.0 1.85; visual mesh filename=file://hailbopp.obj scale=1.0 1.0 1.0

Commit message: Replaced all references to lidar_front/rear to right/left. Parade launch file now contains necessary lidar packages

File: data/hail_bopp.urdf (robot description, URDF)
Before this commit: robot voltron, 8 links, 7 joints
Links:
- removed link lidar_front
- removed link lidar_rear
- added link lidar_left, mass 0.1; collision cylinder length=0.0869 radius=0.05165; visual cylinder length=0.0869 radius=0.05165
- added link lidar_right, mass 0.1; collision cylinder length=0.0869 radius=0.05165; visual cylinder length=0.0869 radius=0.05165
Joints:
- removed joint lidar_front_joint
- removed joint lidar_rear_joint
- added joint lidar_left_joint: type fixed, parent base_link, child lidar_left, origin xyz=-3.5 0.9 1.1 rpy=+0.03 -0.0472 2.65
- added joint lidar_right_joint: type fixed, parent base_link, child lidar_right, origin xyz=0.0 -0.902 0.7876 rpy=-0.015 -0.03 -1.45

Commit message: Fix right lidar tf

File: data/hail_bopp.urdf (robot description, URDF)
Before this commit: robot voltron, 8 links, 7 joints
Joints:
- joint lidar_right_joint: origin xyz=0.0 -0.902 0.7876 rpy=-0.015 -0.03 -1.45 -> xyz=-0.6096 -0.7366 1.8748 rpy=-.20 .20 -.95

Commit message: Re-add core, add to GNSS interface

File: data/hail_bopp.urdf (robot description, URDF)
Before this commit: robot voltron, 8 links, 7 joints
Joints:
- joint gnss_joint: origin xyz=0.0 -0.5 0.5 rpy=0 0 0 -> xyz=-0.5 0.0 1.5 rpy=0 0 0

Commit message: Calibrate LiDARs

File: data/hail_bopp.urdf (robot description, URDF)
Before this commit: robot voltron, 8 links, 7 joints
Links:
- added link model_link; visual mesh filename=file:///navigator/data/hailbopp.stl scale=1.0 1.0 1.0
- link base_link: geometry collision box size=4.37 2.0 1.85
Joints:
- added joint model_joint: type fixed, parent base_link, child model_link, origin xyz=-1.7 -2.3 -0.7 rpy=0 0 -1.570796
- joint lidar_left_joint: origin xyz=-3.5 0.9 1.1 rpy=+0.03 -0.0472 2.65 -> xyz=0.0 0.73 1.5 rpy=0.15 0.2 0.55
- joint lidar_right_joint: origin xyz=-0.6096 -0.7366 1.8748 rpy=-.20 .20 -.95 -> xyz=0.0 -0.73 1.5 rpy=-.20 .20 -.85

Commit message: Multiple changes: - Add LA and GNSS Guardian statuses. - Switch to FastRTPS from CycloneDDS - Add dual_lidar_processing_node

File: data/hail_bopp.urdf (robot description, URDF)
Before this commit: robot voltron, 9 links, 8 joints
Joints:
- joint model_joint: origin xyz=-1.7 -2.3 -0.7 rpy=0 0 -1.570796 -> xyz=-1.2 -2.75 -0.7 rpy=0 0 -1.570796

Commit message: Add LiDAR fusion and calibration, new GNSS interface, and new Guardian messages (#350)
* Remove "epas_translator"

* Delete stale packages

* Create new GNSS package

* Re-add core, add to GNSS interface

* Add pyproj to Dockerfile

* Calibrate LiDARs

* Multiple changes:
- Add LA and GNSS Guardian statuses.
- Switch to FastRTPS from CycloneDDS
- Add dual_lidar_processing_node

* Add .gitignores?

File: data/hail_bopp.urdf (robot description, URDF)
Before this commit: robot voltron, 8 links, 7 joints
Links:
- added link model_link; visual mesh filename=file:///navigator/data/hailbopp.stl scale=1.0 1.0 1.0
- link base_link: geometry collision box size=4.37 2.0 1.85
Joints:
- added joint model_joint: type fixed, parent base_link, child model_link, origin xyz=-1.2 -2.75 -0.7 rpy=0 0 -1.570796
- joint gnss_joint: origin xyz=0.0 -0.5 0.5 rpy=0 0 0 -> xyz=-0.5 0.0 1.5 rpy=0 0 0
- joint lidar_left_joint: origin xyz=-3.5 0.9 1.1 rpy=+0.03 -0.0472 2.65 -> xyz=0.0 0.73 1.5 rpy=0.15 0.2 0.55
- joint lidar_right_joint: origin xyz=-0.6096 -0.7366 1.8748 rpy=-.20 .20 -.95 -> xyz=0.0 -0.73 1.5 rpy=-.20 .20 -.85

Commit message: Added left LiDAR, ground seg, and occ grid

File: data/hail_bopp.urdf (robot description, URDF)
Before this commit: robot voltron, 9 links, 8 joints
Links:
- link model_link: geometry visual mesh filename=file:////home/nova/navigator/data/hailbopp.stl scale=1.0 1.0 1.0

Commit message: Fix lockout in LA interface

File: data/hail_bopp.urdf (robot description, URDF)
Before this commit: robot voltron, 9 links, 8 joints
Joints:
- joint lidar_left_joint: origin xyz=0.0 0.73 1.5 rpy=0.15 0.2 0.55 -> xyz=0.0 0.73 1.8 rpy=0.15 0.2 0.55
- joint lidar_right_joint: origin xyz=0.0 -0.73 1.5 rpy=-.20 .20 -.85 -> xyz=0.0 -0.73 1.8 rpy=-.20 .20 -.85
- joint model_joint: origin xyz=-1.2 -2.75 -0.7 rpy=0 0 -1.570796 -> xyz=-1.2 -2.75 0.0 rpy=0 0 -1.570796

Commit message: Add parameters to MapManager

File: data/hail_bopp.urdf (robot description, URDF)
Before this commit: robot voltron, 9 links, 8 joints
Links:
- link model_link: geometry visual mesh filename=file:////home/wheitman/navigator/data/hailbopp.stl scale=1.0 1.0 1.0

Commit message: Added radar to the urdf file, fixed docker-compose for on-board computer, some updates to the radar processing node and messages

File: data/hail_bopp.urdf (robot description, URDF)
Before this commit: robot voltron, 9 links, 8 joints
Links:
- added link radar
Joints:
- added joint radar_joint: type fixed, parent base_link, child radar, origin xyz=0.61 0.0 0.52 rpy=0 0 0

Commit message: consolidated launch file structure. got radar integrated into rviz

File: data/hail_bopp.urdf (robot description, URDF)
Before this commit: robot voltron, 10 links, 9 joints
Links:
- link model_link: geometry visual mesh filename=file:////navigator/data/hailbopp.stl scale=1.0 1.0 1.0
